Commit message: add OS1-64 (paolo)

File: lidar_description/urdf/example.urdf.xacro (robot description, xacro)
@@ -30,6 +30,6 @@
     </inertial>
   </link>
-  <xacro:include filename="$(find lidar_description)/urdf/VLP-16.urdf.xacro"/>
-  <VLP-16 parent="base_link" name="velodyne" topic="/velodyne_points" hz="10" samples="440" gpu="${gpu}">
+  <xacro:include filename="$(find lidar_description)/urdf/VLP-16.urdf.xacro"/> -->
+ <VLP-16 parent="base_link" name="velodyne" topic="/velodyne_points" hz="10" samples="440" gpu="${gpu}">
     <origin xyz="0 0 0.4" rpy="0 0 0" />
   </VLP-16>
@@ -38,3 +38,7 @@
     <origin xyz="0 0 0.6" rpy="0 0 0" />
   </HDL-32E>
+  <xacro:include filename="$(find lidar_description)/urdf/OS1-64.urdf.xacro"/>
+  <OS1-64 parent="base_link" hz="10" samples="220">
+    <origin xyz="0 0 1.0" rpy="0 0 0" />
+  </OS1-64> -->
 </robot>
