Commit message: tested with VLP-16 and HDL-32E

File: lidar_description/urdf/HDL-32E.urdf.xacro (robot description, xacro)
@@ -18,5 +18,5 @@
       <visual>
         <geometry>
-          <mesh filename="package://velodyne_description/meshes/${name}/${name}_base.dae" />
+          <mesh filename="package://lidar_description/meshes/HDL-32E/HDL-32E_base.dae" />
         </geometry>
       </visual>
@@ -42,5 +42,5 @@
         <origin xyz="0 0 -0.09081" rpy="0 0 0" />
         <geometry>
-          <mesh filename="package://velodyne_description/meshes/${name}/${name}_scan.dae" />
+          <mesh filename="package://lidar_description/meshes/HDL-32E/HDL-32E_scan.dae" />
         </geometry>
       </visual>
@@ -79,5 +79,5 @@
             </noise>
           </ray>
-          <plugin name="gazebo_ros_laser_controller" filename="libgazebo_ros_velodyne_gpu_laser.so">
+          <plugin name="gazebo_ros_laser_controller" filename="libgazebo_ros_lidar_gpu.so">
             <topicName>${topic}</topicName>
             <frameName>${name}</frameName>
@@ -119,5 +119,5 @@
             </noise>
           </ray>
-          <plugin name="gazebo_ros_laser_controller" filename="libgazebo_ros_velodyne_laser.so">
+          <plugin name="gazebo_ros_laser_controller" filename="libgazebo_ros_lidar.so">
             <topicName>${topic}</topicName>
             <frameName>${name}</frameName>

File: lidar_description/urdf/VLP-16.urdf.xacro (robot description, xacro)
@@ -18,10 +18,10 @@
       <visual>
         <geometry>
-          <mesh filename="package://lidar_description/meshes/${name}/${name}_base_1.dae" />
+          <mesh filename="package://lidar_description/meshes/VLP-16/VLP-16_base_1.dae" />
         </geometry>
       </visual>
       <visual>
         <geometry>
-          <mesh filename="package://lidar_description/meshes/${name}/${name}_base_2.dae" />
+          <mesh filename="package://lidar_description/meshes/VLP-16/VLP-16_base_2.dae" />
         </geometry>
       </visual>
@@ -47,5 +47,5 @@
         <origin xyz="0 0 -0.0377" />
         <geometry>
-          <mesh filename="package://lidar_description/${name}/${name}_scan.dae" />
+          <mesh filename="package://lidar_description/meshes/VLP-16/VLP-16_scan.dae" />
         </geometry>
       </visual>

File: lidar_description/urdf/example.urdf.xacro (robot description, xacro)
@@ -34,7 +34,7 @@
     <origin xyz="0 0 0.4" rpy="0 0 0" />
   </VLP-16>
-  <!-- <xacro:include filename="$(find lidar_description)/urdf/HDL-32E.urdf.xacro"/>
+  <xacro:include filename="$(find lidar_description)/urdf/HDL-32E.urdf.xacro"/>
   <HDL-32E parent="base_link" name="velodyne2" topic="/velodyne_points2" hz="10" samples="220" gpu="${gpu}">
     <origin xyz="0 0 0.6" rpy="0 0 0" />
-  </HDL-32E> -->
+  </HDL-32E>
 </robot>
