Commit message: switch to ubuntu 20 - ros noetic

File: lidar_description/urdf/HDL-32E.urdf.xacro (robot description, xacro)
@@ -2,5 +2,5 @@
 <robot xmlns:xacro="http://www.ros.org/wiki/xacro" name="HDL-32E">
   <xacro:property name="M_PI" value="3.1415926535897931" />
-  <xacro:macro name="HDL-32E" params="*origin parent:=base_link name:=velodyne topic:=/velodyne_points hz:=10 lasers:=32 samples:=2187 collision_range:=0.3 min_range:=0.9 max_range:=130.0 noise:=0.008 min_angle:=-${M_PI} max_angle:=${M_PI} gpu:=false">
+  <xacro:macro name="HDL-32E" params="*origin parent:=base_link name:=velodyne topic:=/velodyne_points organize_cloud:=false hz:=10 lasers:=32 samples:=2187 collision_range:=0.3 min_range:=0.9 max_range:=130.0 noise:=0.008 min_angle:=-${M_PI} max_angle:=${M_PI} gpu:=false">
     <joint name="${name}_base_mount_joint" type="fixed">
       <xacro:insert_block name="origin" />
@@ -18,5 +18,5 @@
       <visual>
         <geometry>
-          <mesh filename="package://lidar_description/meshes/HDL-32E/HDL-32E_base.dae" />
+          <mesh filename="package://lidar_description/meshes/HDL32E/HDL32E_base.dae" />
         </geometry>
       </visual>
@@ -42,5 +42,5 @@
         <origin xyz="0 0 -0.09081" rpy="0 0 0" />
         <geometry>
-          <mesh filename="package://lidar_description/meshes/HDL-32E/HDL-32E_scan.dae" />
+          <mesh filename="package://lidar_description/meshes/HDL32E/HDL32E_scan.dae" />
         </geometry>
       </visual>
@@ -82,4 +82,5 @@
             <topicName>${topic}</topicName>
             <frameName>${name}</frameName>
+            <organize_cloud>${organize_cloud}</organize_cloud>
             <min_range>${min_range}</min_range>
             <max_range>${max_range}</max_range>
@@ -122,4 +123,5 @@
             <topicName>${topic}</topicName>
             <frameName>${name}</frameName>
+            <organize_cloud>${organize_cloud}</organize_cloud>
             <min_range>${min_range}</min_range>
             <max_range>${max_range}</max_range>

File: lidar_description/urdf/OS0-128.urdf.xacro (robot description, xacro)
@@ -2,6 +2,6 @@
 <robot xmlns:xacro="http://www.ros.org/wiki/xacro" name="OS0-128">
   <xacro:property name="M_PI" value="3.1415926535897931" />
-  <xacro:macro name="OS0-128" params="*origin parent:=base_link name:=os0_sensor topic:=/os0_cloud_node/points hz:=10 lasers:=128 samples:=512 collision_range:=0.7 min_range:=0.225 max_range:=100.0 noise:=0.008 min_angle:=-${M_PI} max_angle:=${M_PI}">
-    <joint name="mount_joint" type="fixed">
+  <xacro:macro name="OS0-128" params="*origin parent:=base_link name:=os0_sensor topic:=/os0_cloud_node/points organize_cloud:=false hz:=10 lasers:=128 samples:=512 collision_range:=0.7 min_range:=0.225 max_range:=100.0 noise:=0.008 min_angle:=-${M_PI} max_angle:=${M_PI} gpu:=false">
+    <joint name="mount_joint_OS0-128" type="fixed">
       <xacro:insert_block name="origin" />
       <parent link="${parent}"/>
@@ -29,54 +29,103 @@
       </visual>
     </link>
-    <link name="os0_imu" />
-    <link name="os0_lidar" />
-    <joint name="imu_link_joint" type="fixed">
+    <link name="OS0-128_imu" />
+    <link name="OS0-128_lidar" />
+    <joint name="imu_link_joint_OS0-128" type="fixed">
       <parent link="${name}" />
-      <child link="os0_imu" />
+      <child link="OS0-128_imu" />
       <origin xyz="0.006253 -0.011775 0.007645" rpy="0 0 0" />
     </joint>
-    <gazebo reference="os0_imu">
+    <gazebo reference="OS0-128_imu">
     </gazebo>
-    <joint name="lidar_link_joint" type="fixed">
+    <joint name="lidar_link_joint_OS0-128" type="fixed">
       <parent link="${name}" />
-      <child link="os0_lidar" />
+      <child link="OS0-128_lidar" />
       <origin xyz="0.0 0.0 0.03618" rpy="0 0 0" />
     </joint>
-    <!-- Gazebo requires the ouster_gazebo_plugins package -->
-    <gazebo reference="${name}">
-        <sensor type="ray" name="${name}-os0-128">
-          <pose>0 0 0 0 0 0</pose>
-          <visualize>false</visualize>
-          <update_rate>${hz}</update_rate>
-          <ray>
-            <scan>
-              <horizontal>
-                <samples>${samples}</samples>
-                <resolution>1</resolution>
-                <min_angle>${min_angle}</min_angle>
-                <max_angle>${max_angle}</max_angle>
-              </horizontal>
-              <vertical>
-                <samples>${lasers}</samples>
-                <resolution>1</resolution>
-                <min_angle>-${45*M_PI/180.0}</min_angle>
-                <max_angle>${45*M_PI/180.0}</max_angle>
-              </vertical>
-            </scan>
-            <range>
-              <min>${min_range}</min>
-              <max>${max_range}</max>
-              <resolution>0.03</resolution>
-            </range>
-          </ray>
-          <plugin name="gazebo_ros_laser_controller" filename="libgazebo_ros_lidar.so">
-           <topicName>${topic}</topicName>
-            <frameName>${name}</frameName>
-            <min_range>${min_range}</min_range>
-            <max_range>${max_range}</max_range>
-            <gaussianNoise>${noise}</gaussianNoise>
-          </plugin>
-        </sensor>
-    </gazebo>
+ <!-- Gazebo requires the velodyne_gazebo_plugins package -->
+ <gazebo reference="${name}">
+  <xacro:if value="${gpu}">
+    <sensor type="gpu_ray" name="${name}-OS0-128">
+      <pose>0 0 0 0 0 0</pose>
+      <visualize>false</visualize>
+      <update_rate>${hz}</update_rate>
+      <ray>
+        <scan>
+          <horizontal>
+            <samples>${samples}</samples>
+            <resolution>1</resolution>
+            <min_angle>${min_angle}</min_angle>
+            <max_angle>${max_angle}</max_angle>
+          </horizontal>
+          <vertical>
+            <samples>${lasers}</samples>
+            <resolution>1</resolution>
+            <min_angle>-${30.67*M_PI/180.0}</min_angle>
+            <max_angle> ${10.67*M_PI/180.0}</max_angle>
+          </vertical>
+        </scan>
+        <range>
+          <min>${collision_range}</min>
+          <max>${max_range+1}</max>
+          <resolution>0.001</resolution>
+        </range>
+        <noise>
+          <type>gaussian</type>
+          <mean>0.0</mean>
+          <stddev>0.0</stddev>
+        </noise>
+      </ray>
+      <plugin name="gazebo_ros_laser_controller" filename="libgazebo_ros_lidar_gpu.so">
+        <topicName>${topic}</topicName>
+        <frameName>${name}</frameName>
+        <organize_cloud>${organize_cloud}</organize_cloud>
+        <min_range>${min_range}</min_range>
+        <max_range>${max_range}</max_range>
+        <gaussianNoise>${noise}</gaussianNoise>
+      </plugin>
+    </sensor>
+  </xacro:if>
+  <xacro:unless value="${gpu}">
+    <sensor type="ray" name="${name}-OS0-128">
+      <pose>0 0 0 0 0 0</pose>
+      <visualize>false</visualize>
+      <update_rate>${hz}</update_rate>
+      <ray>
+        <scan>
+          <horizontal>
+            <samples>${samples}</samples>
+            <resolution>1</resolution>
+            <min_angle>${min_angle}</min_angle>
+            <max_angle>${max_angle}</max_angle>
+          </horizontal>
+          <vertical>
+            <samples>${lasers}</samples>
+            <resolution>1</resolution>
+            <min_angle>-${45*M_PI/180.0}</min_angle>
+            <max_angle> ${45*M_PI/180.0}</max_angle>
+          </vertical>
+        </scan>
+        <range>
+          <min>${collision_range}</min>
+          <max>${max_range+1}</max>
+          <resolution>0.001</resolution>
+        </range>
+        <noise>
+          <type>gaussian</type>
+          <mean>0.0</mean>
+          <stddev>0.0</stddev>
+        </noise>
+      </ray>
+      <plugin name="gazebo_ros_laser_controller" filename="libgazebo_ros_lidar.so">
+        <topicName>${topic}</topicName>
+        <frameName>${name}</frameName>
+        <organize_cloud>${organize_cloud}</organize_cloud>
+        <min_range>${min_range}</min_range>
+        <max_range>${max_range}</max_range>
+        <gaussianNoise>${noise}</gaussianNoise>
+      </plugin>
+    </sensor>
+  </xacro:unless>
+</gazebo>
   <!-- IMU -->
   <gazebo>
@@ -84,5 +133,5 @@
       <robotNamespace>/</robotNamespace>
       <updateRate>100.0</updateRate>
-      <bodyName>os0_imu</bodyName>
+      <bodyName>OS0-128_imu</bodyName>
       <topicName>/os0_cloud_node/imu</topicName>
       <accelDrift>0.005 0.005 0.005</accelDrift>

File: lidar_description/urdf/OS0-64.urdf.xacro (robot description, xacro)
@@ -2,48 +2,88 @@
 <robot xmlns:xacro="http://www.ros.org/wiki/xacro" name="OS0-64">
   <xacro:property name="M_PI" value="3.1415926535897931" />
-  <xacro:macro name="OS0-64" params="*origin parent:=base_link name:=os0_sensor topic:=/os0_cloud_node/points hz:=10 lasers:=64 samples:=512 collision_range:=0.7 min_range:=0.225 max_range:=100.0 noise:=0.008 min_angle:=-${M_PI} max_angle:=${M_PI}">
-    <joint name="mount_joint" type="fixed">
+  <xacro:macro name="OS0-64" params="*origin parent:=base_link name:=os0_sensor topic:=/os0_cloud_node/points organize_cloud:=false hz:=10 lasers:=64 samples:=512 collision_range:=0.7 min_range:=0.225 max_range:=100.0 noise:=0.008 min_angle:=-${M_PI} max_angle:=${M_PI} gpu:=false">
+    <joint name="mount_joint_OS0-64" type="fixed">
       <xacro:insert_block name="origin" />
-      <parent link="${parent}"/>
-      <child link="${name}"/>
+      <parent link="${parent}" />
+      <child link="${name}" />
     </joint>
     <link name="${name}">
       <inertial>
-         <mass value="0.000000001"/>
-         <origin xyz="0 0 0.0365" rpy="0 0 0" />
-         <inertia ixx="0.000241148" ixy="0" ixz="0"
-          iyy="0.000241148" iyz="0" izz="0.000264"/>
+        <mass value="0.000000001" />
+        <origin xyz="0 0 0.0365" rpy="0 0 0" />
+        <inertia ixx="0.000241148" ixy="0" ixz="0" iyy="0.000241148" iyz="0" izz="0.000264" />
       </inertial>
       <collision name="base_collision">
-         <origin xyz="0 0 0.0365" rpy="0 0 0" />
-         <geometry>
- 	        <cylinder radius="0.04" length="0.073"/>
-         </geometry>
+        <origin xyz="0 0 0.0365" rpy="0 0 0" />
+        <geometry>
+          <cylinder radius="0.04" length="0.073" />
+        </geometry>
       </collision>
       <visual name="base_visual">
-         <origin xyz="0 0 0.0" rpy="0 0 1.5707" />
-         <geometry>
-	         <mesh filename="package://lidar_description/meshes/Ouster/ouster.dae" />
-           <!-- <cylinder length="0.073" radius="0.04" /> -->
-         </geometry>
+        <origin xyz="0 0 0.0" rpy="0 0 1.5707" />
+        <geometry>
+          <mesh filename="package://lidar_description/meshes/Ouster/ouster.dae" />
+          <!-- <cylinder length="0.073" radius="0.04" /> -->
+        </geometry>
       </visual>
     </link>
-    <link name="os0_imu" />
-    <link name="os0_lidar" />
-    <joint name="imu_link_joint" type="fixed">
+    <link name="OS0-64_imu" />
+    <link name="OS0-64_lidar" />
+    <joint name="imu_link_joint_OS0-64" type="fixed">
       <parent link="${name}" />
-      <child link="os0_imu" />
+      <child link="OS0-64_imu" />
       <origin xyz="0.006253 -0.011775 0.007645" rpy="0 0 0" />
     </joint>
-    <gazebo reference="os0_imu">
-    </gazebo>
-    <joint name="lidar_link_joint" type="fixed">
+    <gazebo reference="OS0-64_imu"></gazebo>
+    <joint name="lidar_link_joint_OS0-64" type="fixed">
       <parent link="${name}" />
-      <child link="os0_lidar" />
+      <child link="OS0-64_lidar" />
       <origin xyz="0.0 0.0 0.03618" rpy="0 0 0" />
     </joint>
-    <!-- Gazebo requires the ouster_gazebo_plugins package -->
+    <!-- Gazebo requires the velodyne_gazebo_plugins package -->
     <gazebo reference="${name}">
-        <sensor type="ray" name="${name}-os0-64">
+      <xacro:if value="${gpu}">
+        <sensor type="gpu_ray" name="${name}-OS0-64">
+          <pose>0 0 0 0 0 0</pose>
+          <visualize>false</visualize>
+          <update_rate>${hz}</update_rate>
+          <ray>
+            <scan>
+              <horizontal>
+                <samples>${samples}</samples>
+                <resolution>1</resolution>
+                <min_angle>${min_angle}</min_angle>
+                <max_angle>${max_angle}</max_angle>
+              </horizontal>
+              <vertical>
+                <samples>${lasers}</samples>
+                <resolution>1</resolution>
+                <min_angle>-${30.67*M_PI/180.0}</min_angle>
+                <max_angle> ${10.67*M_PI/180.0}</max_angle>
+              </vertical>
+            </scan>
+            <range>
+              <min>${collision_range}</min>
+              <max>${max_range+1}</max>
+              <resolution>0.001</resolution>
+            </range>
+            <noise>
+              <type>gaussian</type>
+              <mean>0.0</mean>
+              <stddev>0.0</stddev>
+            </noise>
+          </ray>
+          <plugin name="gazebo_ros_laser_controller" filename="libgazebo_ros_lidar_gpu.so">
+            <topicName>${topic}</topicName>
+            <frameName>${name}</frameName>
+            <organize_cloud>${organize_cloud}</organize_cloud>
+            <min_range>${min_range}</min_range>
+            <max_range>${max_range}</max_range>
+            <gaussianNoise>${noise}</gaussianNoise>
+          </plugin>
+        </sensor>
+      </xacro:if>
+      <xacro:unless value="${gpu}">
+        <sensor type="ray" name="${name}-OS0-64">
           <pose>0 0 0 0 0 0</pose>
           <visualize>false</visualize>
@@ -61,16 +101,22 @@
                 <resolution>1</resolution>
                 <min_angle>-${45*M_PI/180.0}</min_angle>
-                <max_angle>${45*M_PI/180.0}</max_angle>
+                <max_angle> ${45*M_PI/180.0}</max_angle>
               </vertical>
             </scan>
             <range>
-              <min>${min_range}</min>
-              <max>${max_range}</max>
-              <resolution>0.03</resolution>
+              <min>${collision_range}</min>
+              <max>${max_range+1}</max>
+              <resolution>0.001</resolution>
             </range>
+            <noise>
+              <type>gaussian</type>
+              <mean>0.0</mean>
+              <stddev>0.0</stddev>
+            </noise>
           </ray>
           <plugin name="gazebo_ros_laser_controller" filename="libgazebo_ros_lidar.so">
-           <topicName>${topic}</topicName>
+            <topicName>${topic}</topicName>
             <frameName>${name}</frameName>
+            <organize_cloud>${organize_cloud}</organize_cloud>
             <min_range>${min_range}</min_range>
             <max_range>${max_range}</max_range>
@@ -78,20 +124,21 @@
           </plugin>
         </sensor>
+      </xacro:unless>
     </gazebo>
-  <!-- IMU -->
-  <gazebo>
-    <plugin name="imu_controller" filename="libhector_gazebo_ros_imu.so">
-      <robotNamespace>/</robotNamespace>
-      <updateRate>100.0</updateRate>
-      <bodyName>os0_imu</bodyName>
-      <topicName>/os0_cloud_node/imu</topicName>
-      <accelDrift>0.005 0.005 0.005</accelDrift>
-      <accelGaussianNoise>0.005 0.005 0.005</accelGaussianNoise>
-      <rateDrift>0.005 0.005 0.005 </rateDrift>
-      <rateGaussianNoise>0.005 0.005 0.005 </rateGaussianNoise>
-      <headingDrift>0.005</headingDrift>
-      <headingGaussianNoise>0.005</headingGaussianNoise>
-    </plugin>
-  </gazebo>
+    <!-- IMU -->
+    <gazebo>
+      <plugin name="imu_controller" filename="libhector_gazebo_ros_imu.so">
+        <robotNamespace>/</robotNamespace>
+        <updateRate>100.0</updateRate>
+        <bodyName>OS0-64_imu</bodyName>
+        <topicName>/os0_cloud_node/imu</topicName>
+        <accelDrift>0.005 0.005 0.005</accelDrift>
+        <accelGaussianNoise>0.005 0.005 0.005</accelGaussianNoise>
+        <rateDrift>0.005 0.005 0.005 </rateDrift>
+        <rateGaussianNoise>0.005 0.005 0.005 </rateGaussianNoise>
+        <headingDrift>0.005</headingDrift>
+        <headingGaussianNoise>0.005</headingGaussianNoise>
+      </plugin>
+    </gazebo>
   </xacro:macro>
 </robot>

File: lidar_description/urdf/OS1-64.urdf.xacro (robot description, xacro)
@@ -28,16 +28,16 @@
       </visual>
     </link>
-    <link name="os1_imu" />
-    <link name="os1_lidar" />
+    <link name="OS1-64_imu" />
+    <link name="OS1-64_lidar" />
     <joint name="imu_link_joint" type="fixed">
       <parent link="${name}" />
-      <child link="os1_imu" />
+      <child link="OS1-64_imu" />
       <origin xyz="0.006253 -0.011775 0.007645" rpy="0 0 0" />
     </joint>
-    <gazebo reference="os1_imu">
+    <gazebo reference="OS1-64_imu">
     </gazebo>
     <joint name="lidar_link_joint" type="fixed">
       <parent link="${name}" />
-      <child link="os1_lidar" />
+      <child link="OS1-64_lidar" />
       <origin xyz="0.0 0.0 0.03618" rpy="0 0 0" />
     </joint>
@@ -120,5 +120,5 @@
         <robotNamespace>/</robotNamespace>
         <updateRate>100.0</updateRate>
-        <bodyName>os1_imu</bodyName>
+        <bodyName>OS1-64_imu</bodyName>
         <topicName>/os1_cloud_node/imu</topicName>
         <accelDrift>0.005 0.005 0.005</accelDrift>

File: lidar_description/urdf/VLP-16.urdf.xacro (robot description, xacro)
@@ -2,5 +2,5 @@
 <robot xmlns:xacro="http://www.ros.org/wiki/xacro" name="VLP-16">
   <xacro:property name="M_PI" value="3.1415926535897931" />
-  <xacro:macro name="VLP-16" params="*origin parent:=base_link name:=velodyne topic:=/velodyne_points hz:=10 lasers:=16 samples:=1875 collision_range:=0.8 min_range:=0.9 max_range:=130.0 noise:=0.008 min_angle:=-${M_PI} max_angle:=${M_PI} gpu:=false">
+  <xacro:macro name="VLP-16" params="*origin parent:=base_link name:=velodyne topic:=/velodyne_points organize_cloud:=false hz:=10 lasers:=16 samples:=1875 collision_range:=0.3 min_range:=0.9 max_range:=130.0 noise:=0.008 min_angle:=-${M_PI} max_angle:=${M_PI} gpu:=false">
     <joint name="${name}_base_mount_joint" type="fixed">
       <xacro:insert_block name="origin" />
@@ -18,10 +18,10 @@
       <visual>
         <geometry>
-          <mesh filename="package://lidar_description/meshes/VLP-16/VLP-16_base_1.dae" />
+          <mesh filename="package://lidar_description/meshes/VLP16/VLP16_base_1.dae" />
         </geometry>
       </visual>
       <visual>
         <geometry>
-          <mesh filename="package://lidar_description/meshes/VLP-16/VLP-16_base_2.dae" />
+          <mesh filename="package://lidar_description/meshes/VLP16/VLP16_base_2.dae" />
         </geometry>
       </visual>
@@ -47,5 +47,5 @@
         <origin xyz="0 0 -0.0377" />
         <geometry>
-          <mesh filename="package://lidar_description/meshes/VLP-16/VLP-16_scan.dae" />
+          <mesh filename="package://lidar_description/meshes/VLP16/VLP16_scan.dae" />
         </geometry>
       </visual>
@@ -87,4 +87,5 @@
             <topicName>${topic}</topicName>
             <frameName>${name}</frameName>
+            <organize_cloud>${organize_cloud}</organize_cloud>
             <min_range>${min_range}</min_range>
             <max_range>${max_range}</max_range>
@@ -127,4 +128,5 @@
             <topicName>${topic}</topicName>
             <frameName>${name}</frameName>
+            <organize_cloud>${organize_cloud}</organize_cloud>
             <min_range>${min_range}</min_range>
             <max_range>${max_range}</max_range>

File: lidar_description/urdf/example.urdf.xacro (robot description, xacro)
@@ -1,15 +1,17 @@
 <?xml version="1.0"?>
 <robot xmlns:xacro="http://www.ros.org/wiki/xacro" name="example">
-  <xacro:arg name="gpu" default="false"/>
+  <xacro:arg name="gpu" default="false" />
   <xacro:property name="gpu" value="$(arg gpu)" />
+  <xacro:arg name="organize_cloud" default="false" />
+  <xacro:property name="organize_cloud" value="$(arg organize_cloud)" />
   <!-- Base Footprint -->
   <link name="base_footprint" />
   <!-- Base Link -->
-  <joint name="footprint" type="fixed" >
-   <parent link="base_footprint" />
+  <joint name="footprint" type="fixed">
+    <parent link="base_footprint" />
     <child link="base_link" />
     <origin xyz="0 0 0.05" rpy="0 0 0" />
   </joint>
-  <link name="base_link" >
+  <link name="base_link">
     <visual>
       <geometry>
@@ -23,22 +25,24 @@
     </collision>
     <inertial>
-      <origin xyz="0 0 0"/>
-      <mass value="10"/>
-      <inertia ixx="3.0" ixy="0.0" ixz="0.0"
-               iyy="3.0" iyz="0.0"
-               izz="3.0" />
+      <origin xyz="0 0 0" />
+      <mass value="10" />
+      <inertia ixx="3.0" ixy="0.0" ixz="0.0" iyy="3.0" iyz="0.0" izz="3.0" />
     </inertial>
   </link>
-  <xacro:include filename="$(find lidar_description)/urdf/VLP-16.urdf.xacro"/> -->
- <VLP-16 parent="base_link" name="velodyne" topic="/velodyne_points" hz="10" samples="440" gpu="${gpu}">
-    <origin xyz="0 0 0.4" rpy="0 0 0" />
-  </VLP-16>
-  <xacro:include filename="$(find lidar_description)/urdf/HDL-32E.urdf.xacro"/>
-  <HDL-32E parent="base_link" name="velodyne2" topic="/velodyne_points2" hz="10" samples="220" gpu="${gpu}">
-    <origin xyz="0 0 0.6" rpy="0 0 0" />
-  </HDL-32E>
-  <xacro:include filename="$(find lidar_description)/urdf/OS1-64.urdf.xacro"/>
-  <OS1-64 parent="base_link" hz="10" samples="220">
-    <origin xyz="0 0 1.0" rpy="0 0 0" />
-  </OS1-64>
+  <xacro:include filename="$(find lidar_description)/urdf/VLP-16.urdf.xacro" />
+  <xacro:VLP-16 parent="base_link" name="velodyne" topic="/velodyne_points" organize_cloud="${organize_cloud}" hz="10" samples="440" gpu="${gpu}">
+    <origin xyz="0.2 0 0.2" rpy="0 0 0" />
+  </xacro:VLP-16>
+  <xacro:include filename="$(find lidar_description)/urdf/HDL-32E.urdf.xacro" />
+  <xacro:HDL-32E parent="base_link" name="velodyne2" topic="/velodyne_points2" organize_cloud="${organize_cloud}" hz="10" samples="220" gpu="${gpu}">
+    <origin xyz="0.2 0.2 0.4" rpy="0 0 0" />
+  </xacro:HDL-32E>
+  <xacro:include filename="$(find lidar_description)/urdf/OS0-64.urdf.xacro" />
+  <xacro:OS0-64 parent="base_link" name="ouster" topic="/ouster_points" organize_cloud="${organize_cloud}" gpu="${gpu}">
+    <origin xyz="-0.2 0 0.6" rpy="0 0 0" />
+  </xacro:OS0-64>
+  <xacro:include filename="$(find lidar_description)/urdf/OS0-128.urdf.xacro" />
+  <xacro:OS0-128 parent="base_link" name="ouster2" topic="/ouster_points2" organize_cloud="${organize_cloud}" gpu="${gpu}">
+    <origin xyz="-0.2 -0.2 0.8" rpy="0 0 0" />
+  </xacro:OS0-128>
 </robot>
