Commit message: add gpu version of OS1-64

File: lidar_description/urdf/OS1-64.urdf.xacro (robot description, xacro)
@@ -2,5 +2,5 @@
 <robot xmlns:xacro="http://www.ros.org/wiki/xacro" name="OS1-64">
   <xacro:property name="M_PI" value="3.1415926535897931" />
-  <xacro:macro name="OS1-64" params="*origin parent:=base_link name:=os1_sensor topic:=/os1_cloud_node/points hz:=10 lasers:=64 samples:=512 collision_range:=0.7 min_range:=0.225 max_range:=100.0 noise:=0.008 min_angle:=-${M_PI} max_angle:=${M_PI}">
+  <xacro:macro name="OS1-64" params="*origin parent:=base_link name:=os1_sensor topic:=/os1_cloud_node/points hz:=10 lasers:=64 samples:=512 collision_range:=0.7 min_range:=0.225 max_range:=100.0 noise:=0.008 min_angle:=-${M_PI} max_angle:=${M_PI} gpu:=false">
     <joint name="mount_joint" type="fixed">
       <xacro:insert_block name="origin" />
@@ -10,21 +10,20 @@
     <link name="${name}">
       <inertial>
-         <mass value="0.000000001"/>
-         <origin xyz="0 0 0.0365" rpy="0 0 0" />
-         <inertia ixx="0.000241148" ixy="0" ixz="0"
-          iyy="0.000241148" iyz="0" izz="0.000264"/>
+        <mass value="0.000000001"/>
+        <origin xyz="0 0 0.0365" rpy="0 0 0" />
+        <inertia ixx="0.000241148" ixy="0" ixz="0" iyy="0.000241148" iyz="0" izz="0.000264"/>
       </inertial>
       <collision name="base_collision">
-         <origin xyz="0 0 0.0365" rpy="0 0 0" />
-         <geometry>
- 	        <cylinder radius="0.04" length="0.073"/>
-         </geometry>
+        <origin xyz="0 0 0.0365" rpy="0 0 0" />
+        <geometry>
+          <cylinder radius="0.04" length="0.073"/>
+        </geometry>
       </collision>
       <visual name="base_visual">
-         <origin xyz="0 0 0.0" rpy="0 0 1.5707" />
-         <geometry>
-	         <mesh filename="package://lidar_description/meshes/Ouster/ouster.dae" />
-           <!-- <cylinder length="0.073" radius="0.04" /> -->
-         </geometry>
+        <origin xyz="0 0 0.0" rpy="0 0 1.5707" />
+        <geometry>
+          <mesh filename="package://lidar_description/meshes/Ouster/ouster.dae" />
+          <!-- <cylinder length="0.073" radius="0.04" /> -->
+        </geometry>
       </visual>
     </link>
@@ -45,4 +44,40 @@
     <!-- Gazebo requires the ouster_gazebo_plugins package -->
     <gazebo reference="${name}">
+      <xacro:if value="${gpu}">
+        <sensor type="gpu_ray" name="${name}-OS1-64">
+          <pose>0 0 0 0 0 0</pose>
+          <visualize>false</visualize>
+          <update_rate>${hz}</update_rate>
+          <ray>
+            <scan>
+              <horizontal>
+                <samples>${samples}</samples>
+                <resolution>1</resolution>
+                <min_angle>${min_angle}</min_angle>
+                <max_angle>${max_angle}</max_angle>
+              </horizontal>
+              <vertical>
+                <samples>${lasers}</samples>
+                <resolution>1</resolution>
+                <min_angle>-${16.611*M_PI/180.0}</min_angle>
+                <max_angle>${16.611*M_PI/180.0}</max_angle>
+              </vertical>
+            </scan>
+            <range>
+              <min>${min_range}</min>
+              <max>${max_range}</max>
+              <resolution>0.03</resolution>
+            </range>
+          </ray>
+          <plugin name="gazebo_ros_laser_controller" filename="libgazebo_ros_lidar_gpu.so">
+            <topicName>${topic}</topicName>
+            <frameName>${name}</frameName>
+            <min_range>${min_range}</min_range>
+            <max_range>${max_range}</max_range>
+            <gaussianNoise>${noise}</gaussianNoise>
+          </plugin>
+        </sensor>
+      </xacro:if>
+      <xacro:unless value="${gpu}">
         <sensor type="ray" name="${name}-OS1-64">
           <pose>0 0 0 0 0 0</pose>
@@ -71,5 +106,5 @@
           </ray>
           <plugin name="gazebo_ros_laser_controller" filename="libgazebo_ros_lidar.so">
-           <topicName>${topic}</topicName>
+            <topicName>${topic}</topicName>
             <frameName>${name}</frameName>
             <min_range>${min_range}</min_range>
@@ -78,20 +113,21 @@
           </plugin>
         </sensor>
+      </xacro:unless>
     </gazebo>
-  <!-- IMU -->
-  <gazebo>
-    <plugin name="imu_controller" filename="libhector_gazebo_ros_imu.so">
-      <robotNamespace>/</robotNamespace>
-      <updateRate>100.0</updateRate>
-      <bodyName>os1_imu</bodyName>
-      <topicName>/os1_cloud_node/imu</topicName>
-      <accelDrift>0.005 0.005 0.005</accelDrift>
-      <accelGaussianNoise>0.005 0.005 0.005</accelGaussianNoise>
-      <rateDrift>0.005 0.005 0.005 </rateDrift>
-      <rateGaussianNoise>0.005 0.005 0.005 </rateGaussianNoise>
-      <headingDrift>0.005</headingDrift>
-      <headingGaussianNoise>0.005</headingGaussianNoise>
-    </plugin>
-  </gazebo>
+    <!-- IMU -->
+    <gazebo>
+      <plugin name="imu_controller" filename="libhector_gazebo_ros_imu.so">
+        <robotNamespace>/</robotNamespace>
+        <updateRate>100.0</updateRate>
+        <bodyName>os1_imu</bodyName>
+        <topicName>/os1_cloud_node/imu</topicName>
+        <accelDrift>0.005 0.005 0.005</accelDrift>
+        <accelGaussianNoise>0.005 0.005 0.005</accelGaussianNoise>
+        <rateDrift>0.005 0.005 0.005 </rateDrift>
+        <rateGaussianNoise>0.005 0.005 0.005 </rateGaussianNoise>
+        <headingDrift>0.005</headingDrift>
+        <headingGaussianNoise>0.005</headingGaussianNoise>
+      </plugin>
+    </gazebo>
   </xacro:macro>
 </robot>

Commit message: fix example for noetic

File: lidar_description/urdf/OS1-64.urdf.xacro (robot description, xacro)
@@ -24,5 +24,4 @@
         <geometry>
           <mesh filename="package://lidar_description/meshes/Ouster/ouster.dae" />
-          <!-- <cylinder length="0.073" radius="0.04" /> -->
         </geometry>
       </visual>

File: lidar_description/urdf/example.urdf.xacro (robot description, xacro)
@@ -31,14 +31,14 @@
   </link>
   <xacro:include filename="$(find lidar_description)/urdf/VLP-16.urdf.xacro"/> -->
- <VLP-16 parent="base_link" name="velodyne" topic="/velodyne_points" hz="10" samples="440" gpu="${gpu}">
+ <xacro:VLP-16 parent="base_link" name="velodyne" topic="/velodyne_points" hz="10" samples="440" gpu="${gpu}">
     <origin xyz="0 0 0.4" rpy="0 0 0" />
-  </VLP-16>
+  </xacro:VLP-16>
   <xacro:include filename="$(find lidar_description)/urdf/HDL-32E.urdf.xacro"/>
-  <HDL-32E parent="base_link" name="velodyne2" topic="/velodyne_points2" hz="10" samples="220" gpu="${gpu}">
+  <xacro:HDL-32E parent="base_link" name="velodyne2" topic="/velodyne_points2" hz="10" samples="220" gpu="${gpu}">
     <origin xyz="0 0 0.6" rpy="0 0 0" />
-  </HDL-32E>
+  </xacro:HDL-32E>
   <xacro:include filename="$(find lidar_description)/urdf/OS1-64.urdf.xacro"/>
-  <OS1-64 parent="base_link" hz="10" samples="220">
+  <xacro:OS1-64 parent="base_link" hz="10" samples="220">
     <origin xyz="0 0 1.0" rpy="0 0 0" />
-  </OS1-64>
+  </xacro:OS1-64>
 </robot>

Commit message: set official params for OS1-64 from datasheet, see rcabg/ouster_example

File: lidar_description/urdf/OS1-64.urdf.xacro (robot description, xacro)
@@ -2,5 +2,5 @@
 <robot xmlns:xacro="http://www.ros.org/wiki/xacro" name="OS1-64">
   <xacro:property name="M_PI" value="3.1415926535897931" />
-  <xacro:macro name="OS1-64" params="*origin parent:=base_link name:=os1_sensor topic:=/os1_cloud_node/points hz:=10 lasers:=64 samples:=512 collision_range:=0.7 min_range:=0.225 max_range:=100.0 noise:=0.008 min_angle:=-${M_PI} max_angle:=${M_PI} gpu:=false">
+  <xacro:macro name="OS1-64" params="*origin parent:=base_link name:=os1_sensor topic_lidar:=/os1_cloud_node/points topic_imu:=/os1_cloud_node/imu hz:=10 lasers:=64 samples:=512 min_range:=0.25 max_range:=75.0 noise:=0.009 min_angle:=-${M_PI} max_angle:=${M_PI} lidar_link:=os1_lidar imu_link:=os1_imu vfov_min:=-.39 vfov_max:=.39">
     <joint name="mount_joint" type="fixed">
       <xacro:insert_block name="origin" />
@@ -59,6 +59,6 @@
                 <samples>${lasers}</samples>
                 <resolution>1</resolution>
-                <min_angle>-${16.611*M_PI/180.0}</min_angle>
-                <max_angle>${16.611*M_PI/180.0}</max_angle>
+                <min_angle>${vfov_min}</min_angle>
+                <max_angle>${vfov_max}</max_angle>
               </vertical>
             </scan>
@@ -70,5 +70,5 @@
           </ray>
           <plugin name="gazebo_ros_laser_controller" filename="libgazebo_ros_lidar_gpu.so">
-            <topicName>${topic}</topicName>
+            <topicName>${topic_lidar}</topicName>
             <frameName>${name}</frameName>
             <min_range>${min_range}</min_range>
@@ -94,6 +94,6 @@
                 <samples>${lasers}</samples>
                 <resolution>1</resolution>
-                <min_angle>-${16.611*M_PI/180.0}</min_angle>
-                <max_angle>${16.611*M_PI/180.0}</max_angle>
+                <min_angle>${vfov_min}</min_angle>
+                <max_angle>${vfov_max}</max_angle>
               </vertical>
             </scan>
@@ -105,5 +105,5 @@
           </ray>
           <plugin name="gazebo_ros_laser_controller" filename="libgazebo_ros_lidar.so">
-            <topicName>${topic}</topicName>
+            <topicName>${topic_lidar}</topicName>
             <frameName>${name}</frameName>
             <min_range>${min_range}</min_range>
@@ -120,5 +120,5 @@
         <updateRate>100.0</updateRate>
         <bodyName>os1_imu</bodyName>
-        <topicName>/os1_cloud_node/imu</topicName>
+        <topicName>${topic_imu}</topicName>
         <accelDrift>0.005 0.005 0.005</accelDrift>
         <accelGaussianNoise>0.005 0.005 0.005</accelGaussianNoise>
