Commit message: added os0 model

File: lidar_description/urdf/OS0-128.urdf.xacro (robot description, xacro)
@@ -1,6 +1,6 @@
 <?xml version="1.0"?>
-<robot xmlns:xacro="http://www.ros.org/wiki/xacro" name="OS1-64">
+<robot xmlns:xacro="http://www.ros.org/wiki/xacro" name="OS0-128">
   <xacro:property name="M_PI" value="3.1415926535897931" />
-  <xacro:macro name="OS1-64" params="*origin parent:=base_link name:=os1_sensor topic:=/os1_cloud_node/points hz:=10 lasers:=64 samples:=512 collision_range:=0.7 min_range:=0.225 max_range:=100.0 noise:=0.008 min_angle:=-${M_PI} max_angle:=${M_PI}">
+  <xacro:macro name="OS0-128" params="*origin parent:=base_link name:=os0_sensor topic:=/os0_cloud_node/points hz:=10 lasers:=128 samples:=512 collision_range:=0.7 min_range:=0.225 max_range:=100.0 noise:=0.008 min_angle:=-${M_PI} max_angle:=${M_PI}">
     <joint name="mount_joint" type="fixed">
       <xacro:insert_block name="origin" />
@@ -29,21 +29,21 @@
       </visual>
     </link>
-    <link name="os1_imu" />
-    <link name="os1_lidar" />
+    <link name="os0_imu" />
+    <link name="os0_lidar" />
     <joint name="imu_link_joint" type="fixed">
       <parent link="${name}" />
-      <child link="os1_imu" />
+      <child link="os0_imu" />
       <origin xyz="0.006253 -0.011775 0.007645" rpy="0 0 0" />
     </joint>
-    <gazebo reference="os1_imu">
+    <gazebo reference="os0_imu">
     </gazebo>
     <joint name="lidar_link_joint" type="fixed">
       <parent link="${name}" />
-      <child link="os1_lidar" />
+      <child link="os0_lidar" />
       <origin xyz="0.0 0.0 0.03618" rpy="0 0 0" />
     </joint>
     <!-- Gazebo requires the ouster_gazebo_plugins package -->
     <gazebo reference="${name}">
-        <sensor type="ray" name="${name}-OS1-64">
+        <sensor type="ray" name="${name}-os0-128">
           <pose>0 0 0 0 0 0</pose>
           <visualize>false</visualize>
@@ -60,6 +60,6 @@
                 <samples>${lasers}</samples>
                 <resolution>1</resolution>
-                <min_angle>-${16.611*M_PI/180.0}</min_angle>
-                <max_angle>${16.611*M_PI/180.0}</max_angle>
+                <min_angle>-${45*M_PI/180.0}</min_angle>
+                <max_angle>${45*M_PI/180.0}</max_angle>
               </vertical>
             </scan>
@@ -84,6 +84,6 @@
       <robotNamespace>/</robotNamespace>
       <updateRate>100.0</updateRate>
-      <bodyName>os1_imu</bodyName>
-      <topicName>/os1_cloud_node/imu</topicName>
+      <bodyName>os0_imu</bodyName>
+      <topicName>/os0_cloud_node/imu</topicName>
       <accelDrift>0.005 0.005 0.005</accelDrift>
       <accelGaussianNoise>0.005 0.005 0.005</accelGaussianNoise>

Commit message: Updated code for cohort_icra
Signed-off-by: Mihir Kulkarni <mihirk284@gmail.com>

File: lidar_description/urdf/OS0-128.urdf.xacro (robot description, xacro)
@@ -2,5 +2,5 @@
 <robot xmlns:xacro="http://www.ros.org/wiki/xacro" name="OS0-128">
   <xacro:property name="M_PI" value="3.1415926535897931" />
-  <xacro:macro name="OS0-128" params="*origin parent:=base_link name:=os0_sensor topic:=/os0_cloud_node/points hz:=10 lasers:=128 samples:=512 collision_range:=0.7 min_range:=0.225 max_range:=100.0 noise:=0.008 min_angle:=-${M_PI} max_angle:=${M_PI}">
+  <xacro:macro name="OS0-128" params="*origin parent:=base_link name:=os0_sensor topic:=/os0_cloud_node/points hz:=10 lasers:=128 samples:=256 collision_range:=0.7 min_range:=0.225 max_range:=100.0 noise:=0.008 min_angle:=-${M_PI} max_angle:=${M_PI}">
     <joint name="mount_joint" type="fixed">
       <xacro:insert_block name="origin" />

File: lidar_description/urdf/OS1-64.urdf.xacro (robot description, xacro)
@@ -2,5 +2,5 @@
 <robot xmlns:xacro="http://www.ros.org/wiki/xacro" name="OS1-64">
   <xacro:property name="M_PI" value="3.1415926535897931" />
-  <xacro:macro name="OS1-64" params="*origin parent:=base_link name:=os1_sensor topic:=/os1_cloud_node/points hz:=10 lasers:=64 samples:=512 collision_range:=0.7 min_range:=0.225 max_range:=100.0 noise:=0.008 min_angle:=-${M_PI} max_angle:=${M_PI} gpu:=false">
+  <xacro:macro name="OS1-64" params="*origin parent:=base_link name:=os1_sensor topic:=/os1_cloud_node/points hz:=10 lasers:=64 samples:=512 collision_range:=0.7 min_range:=0.225 max_range:=100.0 noise:=0.008 min_angle:=-${M_PI} max_angle:=${M_PI} gpu:=false vertical_angle:=16.611">
     <joint name="mount_joint" type="fixed">
       <xacro:insert_block name="origin" />
@@ -60,6 +60,6 @@
                 <samples>${lasers}</samples>
                 <resolution>1</resolution>
-                <min_angle>-${16.611*M_PI/180.0}</min_angle>
-                <max_angle>${16.611*M_PI/180.0}</max_angle>
+                <min_angle>-${vertical_angle*M_PI/180.0}</min_angle>
+                <max_angle>${vertical_angle*M_PI/180.0}</max_angle>
               </vertical>
             </scan>
@@ -95,6 +95,6 @@
                 <samples>${lasers}</samples>
                 <resolution>1</resolution>
-                <min_angle>-${16.611*M_PI/180.0}</min_angle>
-                <max_angle>${16.611*M_PI/180.0}</max_angle>
+                <min_angle>-${vertical_angle}*M_PI/180.0}</min_angle>
+                <max_angle>${vertical_angle}*M_PI/180.0}</max_angle>
               </vertical>
             </scan>

File: lidar_description/urdf/VLP-16.urdf.xacro (robot description, xacro)
@@ -10,5 +10,5 @@
     <link name="${name}_base_link">
       <inertial>
-        <mass value="0.83"/>
+        <mass value="0.000000001"/>
         <origin xyz="0 0 0.03585"/>
         <inertia ixx="${(0.83 * (3.0*0.0516*0.0516 + 0.0717*0.0717)) / 12.0}" ixy="0" ixz="0"

Commit message: Added function for organized cloud

File: lidar_description/urdf/OS0-128.urdf.xacro (robot description, xacro)
@@ -2,5 +2,5 @@
 <robot xmlns:xacro="http://www.ros.org/wiki/xacro" name="OS0-128">
   <xacro:property name="M_PI" value="3.1415926535897931" />
-  <xacro:macro name="OS0-128" params="*origin parent:=base_link name:=os0_sensor topic:=/os0_cloud_node/points hz:=10 lasers:=128 samples:=512 collision_range:=0.7 min_range:=0.225 max_range:=100.0 noise:=0.008 min_angle:=-${M_PI} max_angle:=${M_PI}">
+  <xacro:macro name="OS0-128" params="*origin parent:=base_link name:=os0_sensor organize_cloud:=false topic:=/os0_cloud_node/points hz:=10 lasers:=128 samples:=512 collision_range:=0.7 min_range:=0.225 max_range:=100.0 noise:=0.008 min_angle:=-${M_PI} max_angle:=${M_PI} gpu:=false">
     <joint name="mount_joint" type="fixed">
       <xacro:insert_block name="origin" />
@@ -45,4 +45,43 @@
     <!-- Gazebo requires the ouster_gazebo_plugins package -->
     <gazebo reference="${name}">
+      <xacro:if value="${gpu}">
+        <sensor type="gpu_ray" name="${name}-os0-128">
+          <pose>0 0 0 0 0 0</pose>
+          <visualize>false</visualize>
+          <update_rate>${hz}</update_rate>
+          <ray>
+            <scan>
+              <horizontal>
+                <samples>${samples}</samples>
+                <resolution>1</resolution>
+                <min_angle>${min_angle}</min_angle>
+                <max_angle>${max_angle}</max_angle>
+              </horizontal>
+              <vertical>
+                <samples>${lasers}</samples>
+                <resolution>1</resolution>
+                <min_angle>-${45*M_PI/180.0}</min_angle>
+                <max_angle>${45*M_PI/180.0}</max_angle>
+                <!-- <min_angle>-${75*M_PI/180.0}</min_angle>
+                <max_angle>${75*M_PI/180.0}</max_angle> -->
+              </vertical>
+            </scan>
+            <range>
+              <min>${min_range}</min>
+              <max>${max_range}</max>
+              <resolution>0.03</resolution>
+            </range>
+          </ray>
+          <plugin name="gazebo_ros_laser_controller" filename="libgazebo_ros_lidar_gpu.so">
+           <topicName>${topic}</topicName>
+            <frameName>${name}</frameName>
+            <organize_cloud>${organize_cloud}</organize_cloud>
+            <min_range>${min_range}</min_range>
+            <max_range>${max_range}</max_range>
+            <gaussianNoise>${noise}</gaussianNoise>
+          </plugin>
+        </sensor>
+      </xacro:if>
+      <xacro:unless value="${gpu}">
         <sensor type="ray" name="${name}-os0-128">
           <pose>0 0 0 0 0 0</pose>
@@ -73,4 +112,5 @@
            <topicName>${topic}</topicName>
             <frameName>${name}</frameName>
+            <organize_cloud>${organize_cloud}</organize_cloud>
             <min_range>${min_range}</min_range>
             <max_range>${max_range}</max_range>
@@ -78,4 +118,5 @@
           </plugin>
         </sensor>
+      </xacro:unless>
     </gazebo>
   <!-- IMU -->

File: lidar_description/urdf/OS1-64.urdf.xacro (robot description, xacro)
@@ -2,5 +2,5 @@
 <robot xmlns:xacro="http://www.ros.org/wiki/xacro" name="OS1-64">
   <xacro:property name="M_PI" value="3.1415926535897931" />
-  <xacro:macro name="OS1-64" params="*origin parent:=base_link name:=os1_sensor topic:=/os1_cloud_node/points hz:=10 lasers:=64 samples:=512 collision_range:=0.7 min_range:=0.225 max_range:=100.0 noise:=0.008 min_angle:=-${M_PI} max_angle:=${M_PI} gpu:=false">
+  <xacro:macro name="OS1-64" params="*origin parent:=base_link name:=os1_sensor topic:=/os1_cloud_node/points hz:=10 lasers:=64 samples:=512 collision_range:=0.7 min_range:=0.225 max_range:=100.0 noise:=0.008 min_angle:=-${M_PI} max_angle:=${M_PI} gpu:=false organize_cloud:=true">
     <joint name="mount_joint" type="fixed">
       <xacro:insert_block name="origin" />
@@ -60,6 +60,8 @@
                 <samples>${lasers}</samples>
                 <resolution>1</resolution>
-                <min_angle>-${16.611*M_PI/180.0}</min_angle>
-                <max_angle>${16.611*M_PI/180.0}</max_angle>
+                <!-- <min_angle>-${16.611*M_PI/180.0}</min_angle>
+                <max_angle>${16.611*M_PI/180.0}</max_angle> -->
+                <min_angle>-${7.0*M_PI/180.0}</min_angle>
+                <max_angle>${45.0*M_PI/180.0}</max_angle>
               </vertical>
             </scan>
@@ -75,4 +77,5 @@
             <min_range>${min_range}</min_range>
             <max_range>${max_range}</max_range>
+            <organize_cloud>${organize_cloud}</organize_cloud>
             <gaussianNoise>${noise}</gaussianNoise>
           </plugin>
@@ -110,4 +113,5 @@
             <min_range>${min_range}</min_range>
             <max_range>${max_range}</max_range>
+            <organize_cloud>${organize_cloud}</organize_cloud>
             <gaussianNoise>${noise}</gaussianNoise>
           </plugin>
